File: drawing.kicad_v3.0_pcb.kicad_pcb (KiCad board)
At the start: 2 copper layers, 93 x 65 mm, 40 parts, among them IC1 DW01A-G, J1 Micro USB Chargeport, J2 Prog headers, J3 128x32 I2C OLED, J4 TP4056, J5 MK-12C02, J6 Conn_01x02, Q1 FS8205, U1 HT7333-SOT89, U2 ESP-12E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

Commit message: Updated charging circuit
Parts:
- removed REF**: OSHW, user-footprints:OSHW
- turned C4 to -90 degrees
Connections:
- net /+5V renamed Net-(C2-Pad2)
- C4 pad 1: /Batt- -> Net-(C4-Pad1)
- C4 pad 2: Net-(C4-Pad2) -> GND
- IC1 pad 5: Net-(C4-Pad2) -> Net-(C4-Pad1)
- IC1 pad 6: /Batt- -> GND
- J1 pad 4: GND -> unconnected-(J1-Pad4)
- J6 pad 1: /Batt+ -> GND
- J6 pad 2: /Batt- -> /Batt+
- Q1 pad 1: unconnected-(Q1-Pad1) -> GND
- Q1 pad 2: GND -> unconnected-(Q1-Pad2)
- Q1 pad 3: unconnected-(Q1-Pad3) -> GND
- Q1 pad 5: /Batt- -> unconnected-(Q1-Pad5)
- R10 pad 2: Net-(J4-Pad6) -> Net-(J4-Pad7)
- R12 pad 1: Net-(J4-Pad7) -> Net-(J4-Pad6)
- R14 pad 2: Net-(C4-Pad2) -> Net-(C4-Pad1)
Routing:
- net /Batt-: track 77.6 -> 0.00 mm, vias 2 -> 0
- net Net-(C4-Pad2): track 28.2 -> 0.00 mm
- net Net-(C4-Pad1): track 0.00 -> 18.1 mm
- net Net-(J4-Pad7): track 9.24 -> 5.11 mm
- net +3V3: track 160.2 -> 157.0 mm
- net /Batt+: track 76.3 -> 78.8 mm
- net GND: track 96.5 -> 94.5 mm, vias 1 -> 8
- net Net-(J4-Pad6): track 4.58 -> 5.62 mm

Commit message: Fixed charging circuit in v3.0
Parts:
- J2: value Prog headers -> Conn_01x03; footprint Connector_PinSocket_2.54mm:PinSocket_1x04_P2.54mm_Horizontal -> Connector_PinSocket_2.54mm:PinSocket_1x03_P2.54mm_Horizontal
Connections:
- J2 pad 1: /RX -> GND
- J2 pad 2: /TX -> /RX
- J2 pad 3: GND -> /TX
Routing:
- net /RX: track 42.1 -> 43.8 mm
- net /TX: track 40.1 -> 41.4 mm
- net GND: vias 8 -> 3
Other:
- board text removed: "DTR"

Commit message: Fixed esp8266 programming circuit in v3.0
Parts:
- added REF**: OSHW, user-footprints:OSHW, B.Cu at (194.2, 66.1)
- added S3: PTS645SM43SMTR92_LFS, digikey-footprints:Switch_Tactile_SMD_6x6mm_PTS645, B.Cu at (165.1, 107.8)
- S2: moved to B.Cu
- moved S2 22.7 mm to (153.6, 107.8), turned to 0 degrees
Connections:
- net /DTR renamed Net-(U2-Pad18)
- R6 pad 2: Net-(R6-Pad2) -> Net-(S2-Pad1)
- R8 pad 1: Net-(R8-Pad1) -> Net-(U2-Pad16)
- S2 pad 1: GND -> Net-(S2-Pad1)
- S2 pad 2: GND -> Net-(S2-Pad1)
- S2 pad 3: Net-(R6-Pad2) -> GND
- S2 pad 4: Net-(R6-Pad2) -> GND
- U2 pad 1: Net-(R6-Pad2) -> Net-(S2-Pad1)
- U2 pad 16: GND -> Net-(U2-Pad16)
- U2 pad 4: Net-(R8-Pad1) -> unconnected-(U2-Pad4)
Routing:
- net Net-(R6-Pad2): track 78.3 -> 0.00 mm, vias 1 -> 0
- net Net-(S2-Pad1): track 0.00 -> 51.6 mm, vias 0 -> 2
- net Net-(U2-Pad16): track 0.00 -> 24.5 mm, vias 0 -> 2
- net Net-(U2-Pad18): track 63.5 -> 81.8 mm
- net GND: track 94.5 -> 83.2 mm
- net Net-(R8-Pad1): track 4.61 -> 0.00 mm
Other:
- board text added: "Program"
