File: drawing.kicad_v3.1_pcb.kicad_pcb (KiCad board)
At the start: 2 copper layers, 93 x 65 mm, 42 parts, among them IC1 DW01A-G, J1 Micro USB Chargeport, J2 Conn_01x03, J3 128x32 I2C OLED, J4 TP4056, J5 MK-12C02, J6 Conn_01x02, Q1 FS8205, U1 HT7333-SOT89, U2 ESP-12E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

Commit message: Run from 18650 and fixed HT7333 circuit
Parts:
- added REF**: OSHW, user-footprints:OSHW, B.Cu at (194.1, 65.8)
Other:
- board text added: "v3.1"
- board text removed: "v3.0"
